File: 3dfx-sli-1slot/3dfx-sli-1slot.kicad_pcb (KiCad board)
At the start: 4 copper layers, 44.2 x 26.4 mm, 3 parts, among them J1 3DFX-SLI, J2 3DFX-SLI

Commit message: Add files via upload
Other:
- board text added: "3Dfx SLI Bridge (single slot spacing)"
- board text removed: "3Dfx SLI Bridge (single slot spaing)"
Changed lines of the file:
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@@
     (descr "Through hole straight pin header, 2x17, 2.54mm pitch, double rows")
     (tags "Through hole pin header THT 2x17 2.54mm double row")
-    (fp_text reference J1 (at 1.27 2.54 90) (layer B.SilkS)
+    (fp_text reference J1 (at 1.27 2.54 90) (layer B.SilkS) hide
       (effects (font (size 1 1) (thickness 0.15)) (justify mirror))
     )
@@
     (descr "Through hole straight pin header, 2x17, 2.54mm pitch, double rows")
     (tags "Through hole pin header THT 2x17 2.54mm double row")
-    (fp_text reference J2 (at 1.27 2.667 90) (layer B.SilkS)
+    (fp_text reference J2 (at 1.27 2.667 90) (layer B.SilkS) hide
       (effects (font (size 1 1) (thickness 0.15)) (justify mirror))
     )
@@
     )
   )
-  (gr_text JLCJLCJLCJLC (at 153.035 91.567) (layer B.SilkS)
+  (gr_text JLCJLCJLCJLC (at 152.019 91.44) (layer B.SilkS)
     (effects (font (size 1 1) (thickness 0.15)) (justify mirror))
   )
@@
     (effects (font (size 1 1) (thickness 0.15)) (justify mirror))
   )
-  (gr_text "3Dfx SLI Bridge (single slot spaing)" (at 159.512 104.648) (layer B.SilkS)
-    (effects (font (size 1 1) (thickness 0.15)) (justify mirror))
-  )
+  (gr_text "3Dfx SLI Bridge (single slot spacing)" (at 159.131 104.648) (layer B.SilkS)
+    (effects (font (size 1 1) (thickness 0.15)) (justify mirror))
+  )
